File: BMP.kicad_sch (KiCad schematic)
At the start: 29 parts, among them CN1 USB_B_Mini, J1 Conn_01x04_Pin, J2 Conn_02x05_Odd_Even, Q1 IRLML5203, SW1 SW_Push, SW2 SW_Push, U1 STM32F103CBTx, U2 TXS0108EPW, Y1 8MHz

Commit message: schematic done
Parts:
- added C1, C2: 1uF, Capacitor_SMD:C_0805_2012Metric_Pad1.18x1.45mm_HandSolder, symbol Device:C
- added C3, C4, C5: 100nF, Capacitor_SMD:C_0805_2012Metric_Pad1.18x1.45mm_HandSolder, symbol Device:C
- added U3: TLV70033_SOT23-5, Package_TO_SOT_SMD:SOT-23-5, symbol Regulator_Linear:TLV70033_SOT23-5
- C7: footprint (none) -> Capacitor_SMD:C_0603_1608Metric_Pad1.08x0.95mm_HandSolder
- D1, D2, D3, D4: footprint (none) -> Resistor_SMD:R_0603_1608Metric_Pad0.98x0.95mm_HandSolder
- J2: footprint (none) -> Connector_IDC:IDC-Header_2x05_P2.54mm_Vertical
Connections:
- net +3.3V: now also Q1.2 (S), C2.2, C3.2, C4.2, C5.2, U3.5 (OUT)
- net +5V: now also C1.2, U3.1 (IN), U3.3 (EN)
- net GND: now also J2.3 (Pin_3), J2.5 (Pin_5), J2.9 (Pin_9), C1.1, C2.1, C3.1, C4.1, C5.1, U3.2 (GND)
- net LED0: now also U1.20 (PB2)
- net PWR_BR: now also U1.19 (PB1)
- net RXD: no longer J1.2 (Pin_2), U1.30 (PA9), U1.37 (PA14)
- net TPWR: now also J2.1 (Pin_1), Q1.3 (D), U2.10 (OE), U2.2 (VCCA)
- net TARGET_POWER_ADC: now reaches C6.2, R6.2, R8.2, U1.18 (PB0)
- new net TXD: J1.2 (Pin_2), U1.30 (PA9), U1.37 (PA14)
- now unconnected: U2.1 (A1)
- no-connect marks 8 -> 19

Commit message: 15032023
Parts:
- SW1, SW2: footprint (none) -> Custom PADs:BMP_SWITCH_2PIN
Changed lines of the file:
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@@
       (effects (font (size 1.27 1.27)) (justify right) hide)
     )
-    (property "Footprint" "" (at 118.11 25.4 0)
+    (property "Footprint" "Custom PADs:BMP_SWITCH_2PIN" (at 118.11 25.4 0)
       (effects (font (size 1.27 1.27)) hide)
     )
@@
       (effects (font (size 1.27 1.27)) (justify right) hide)
     )
-    (property "Footprint" "" (at 99.06 78.74 0)
-      (effects (font (size 1.27 1.27)) hide)
-    )
+    (property "Footprint" "Custom PADs:BMP_SWITCH_2PIN" (at 99.06 78.74 0)
+      (effects (font (size 1.27 1.27)) hide)
+    )

Commit message: beta PCB complete
Parts:
- C3, C4, C5, C6: footprint Capacitor_SMD:C_0805_2012Metric_Pad1.18x1.45mm_HandSolder -> Capacitor_SMD:C_0603_1608Metric_Pad1.08x0.95mm_HandSolder
- R3: value 220 -> 1K5
Changed lines of the file:
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@@
       (effects (font (size 1.27 1.27)) (justify right))
     )
-    (property "Footprint" "Capacitor_SMD:C_0805_2012Metric_Pad1.18x1.45mm_HandSolder" (at 93.0148 57.15 0)
+    (property "Footprint" "Capacitor_SMD:C_0603_1608Metric_Pad1.08x0.95mm_HandSolder" (at 93.0148 57.15 0)
       (effects (font (size 1.27 1.27)) hide)
     )
@@
       (effects (font (size 1.27 1.27)) (justify right))
     )
-    (property "Footprint" "Capacitor_SMD:C_0805_2012Metric_Pad1.18x1.45mm_HandSolder" (at 173.0248 135.89 0)
+    (property "Footprint" "Capacitor_SMD:C_0603_1608Metric_Pad1.08x0.95mm_HandSolder" (at 173.0248 135.89 0)
       (effects (font (size 1.27 1.27)) hide)
     )
@@
       (effects (font (size 1.27 1.27)))
     )
-    (property "Value" "220" (at 193.04 43.18 90)
+    (property "Value" "1K5" (at 193.04 43.18 90)
       (effects (font (size 1.27 1.27)))
     )
@@
       (effects (font (size 1.27 1.27)) (justify right))
     )
-    (property "Footprint" "Capacitor_SMD:C_0805_2012Metric_Pad1.18x1.45mm_HandSolder" (at 183.1848 135.89 0)
+    (property "Footprint" "Capacitor_SMD:C_0603_1608Metric_Pad1.08x0.95mm_HandSolder" (at 183.1848 135.89 0)
       (effects (font (size 1.27 1.27)) hide)
     )
@@
       (effects (font (size 1.27 1.27)) (justify right))
     )
-    (property "Footprint" "Capacitor_SMD:C_0805_2012Metric_Pad1.18x1.45mm_HandSolder" (at 192.0748 135.89 0)
-      (effects (font (size 1.27 1.27)) hide)
-    )
+    (property "Footprint" "Capacitor_SMD:C_0603_1608Metric_Pad1.08x0.95mm_HandSolder" (at 192.0748 135.89 0)
+      (effects (font (size 1.27 1.27)) hide)
+    )
